Commit message: update 2025

File: moveit2_ur3e_config/config/ur3e_bot.ros2_control.xacro (robot description, xacro)
@@ -7,7 +7,7 @@
                 <!-- By default, set up controllers for simulation. This won't work on real hardware -->
                 <!-- plugin>mock_components/GenericSystem</plugin -->
-                <plugin>topic_based_ros2_control/TopicBasedSystem</plugin>
+                <!-- <plugin>topic_based_ros2_control/TopicBasedSystem</plugin>
                 <param name="joint_commands_topic">/isaac_joint_commands</param>
-                <param name="joint_states_topic">/isaac_joint_states</param>
+                <param name="joint_states_topic">/isaac_joint_states</param> -->
             </hardware>
             <joint name="shoulder_pan_joint">

File: moveit2_ur3e_config/config/ur3e_bot.urdf (robot description, URDF)
Before this commit: robot ur3e_bot, 33 links, 32 joints
Joints:
- joint robotiq_coupler_joint: origin xyz=0 0 0.004 rpy=0 0 -1.5707963267948966 -> xyz=0 0 0.004 rpy=0 0 0
- joint ur3e_robotiq_2f_140_joint: origin xyz=0 0 0.004 rpy=0 0 -1.5707963267948966 -> xyz=0 0 0.004 rpy=0 0 0

File: ur3e_robot_description/urdf/ur3e/robot.urdf.xacro (robot description, xacro)
@@ -29,5 +29,5 @@
     </joint>
     <joint name="ur3e_robotiq_2f_140_joint" type="fixed">
-      <origin xyz="0 0 0.004" rpy="0 0 ${-pi/2.0}" />
+      <origin xyz="0 0 0.004" rpy="0 0 0" />
       <parent link="robotiq_coupler"/>
       <child link="robotiq_arg2f_base_link"/>
